File: CHeepCore/CHeepCore.kicad_sch (KiCad schematic)
At the start: 8 parts, among them J101 Conn_01x10, J102 Conn_01x10, U101 CH32V003FxUx, Y101 Crystal_GND24

Commit message: Added USB to smd pad
USB smd pads added on the back
Parts:
- added J103: USB, Connector_PinHeader_1.00mm:PinHeader_2x01_P1.00mm_Vertical_SMD, symbol Connector_Generic:Conn_01x02
Connections:
- net USB with LDO/D+: now also J103.1 (Pin_1)
- net USB with LDO/D-: now also J103.2 (Pin_2)
- no-connect marks 7 -> 5

Commit message: Changed to TSSOP Footprint
Changed to WCH CH32V003F4P6
Parts:
- removed U101: CH32V003FxUx, Package_DFN_QFN:QFN-20-1EP_3x3mm_P0.4mm_EP1.65x1.65mm, symbol MCU_WCH_CH32V0:CH32V003FxUx
- added U101: CH32V003FxPx, Package_SO:TSSOP-20_4.4x6.5mm_P0.65mm, symbol MCU_WCH_CH32V0:CH32V003FxPx
Connections:
- net GND: now also U101.7 (VSS)
- net PC0: now also U101.10 (PC0)
- net PC1: now also U101.11 (PC1)
- net PC2: now also U101.12 (PC2)
- net PC3: now also U101.13 (PC3)
- net PC4: now also U101.14 (PC4)
- net PC5: now also U101.15 (PC5)
- net PC6: now also U101.16 (PC6)
- net PC7: now also U101.17 (PC7)
- net PD0: now also U101.8 (PD0)
- net PD1: now also U101.18 (PD1)
- net PD2: now also U101.19 (PD2)
- net PD3: now also U101.20 (PD3)
- net PD4: now also U101.1 (PD4)
- net PD5: now also U101.2 (PD5)
- net PD6: now also U101.3 (PD6)
- net PD7: now also U101.4 (PD7)
- net at C103.1, Y101.1: now also U101.5 (PA1)
- net at C101.1, JP101.2 (C): now also U101.9 (VDD)
- net at C102.1, Y101.3: now also U101.6 (PA2)
Changed lines of the file:
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@@
-	)
-	(symbol
-		(lib_id "MCU_WCH_CH32V0:CH32V003FxUx")
-		(at 123.19 105.41 0)
-		(unit 1)
-		(exclude_from_sim no)
-		(in_bom yes)
-		(on_board yes)
-		(dnp no)
-		(fields_autoplaced yes)
-		(property "Reference" "U101"
-			(at 125.4551 85.09 0)
-			(effects
-				(font
-					(size 1.27 1.27)
-				)
-				(justify left)
-			)
-		)
-		(property "Value" "CH32V003FxUx"
-			(at 125.4551 87.63 0)
-			(effects
-				(font
-					(size 1.27 1.27)
-				)
-				(justify left)
-			)
-		)
-		(property "Footprint" "Package_DFN_QFN:QFN-20-1EP_3x3mm_P0.4mm_EP1.65x1.65mm"
-			(at 121.92 105.41 0)
-			(effects
-				(font
-					(size 1.27 1.27)
-				)
-				(hide yes)
-			)
-		)
-		(property "Datasheet" "https://www.wch-ic.com/products/CH32V003.html"
-			(at 121.92 105.41 0)
-			(effects
-				(font
-					(size 1.27 1.27)
-				)
-				(hide yes)
-			)
-		)
-		(property "Description" "CH32V003 series are industrial-grade general-purpose microcontrollers designed based on 32-bit RISC-V instruction set and architecture. It adopts QingKe V2A core, RV32EC instruction set, and supports 2 levels of interrupt nesting. The series are mounted with rich peripheral interfaces and function modules. Its internal organizational structure meets the low-cost and low-power embedded application scenarios."
-			(at 123.19 105.41 0)
-			(effects
-				(font
-					(size 1.27 1.27)
-				)
-				(hide yes)
-			)
-		)
-		(property "LCSC" "https://www.lcsc.com/product-detail/C5299908.html?s_z=n_CH32v003"
-			(at 123.19 105.41 0)
-			(effects
-				(font
-					(size 1.27 1.27)
-				)
-				(hide yes)
-			)
-		)
-		(property "Price @ 1000" "0.1599 €"
-			(at 123.19 105.41 0)
-			(effects
-				(font
-					(size 1.27 1.27)
-				)
-				(hide yes)
-			)
-		)
-		(property "DigiKey" ""
-			(at 123.19 105.41 0)
-			(effects
-				(font
-					(size 1.27 1.27)
-				)
-				(hide yes)
-			)
-		)
-		(pin "17"
-		)
-		(pin "8"
-		)
-		(pin "6"
-		)
-		(pin "21"
-		)
-		(pin "15"
-		)
-		(pin "7"
-		)
-		(pin "9"
-		)
-		(pin "10"
-		)
-		(pin "11"
-		)
-		(pin "12"
-		)
-		(pin "13"
-		)
-		(pin "5"
-		)
-		(pin "14"
-		)
-		(pin "4"
-		)
-		(pin "16"
-		)
-		(pin "18"
-		)
-		(pin "19"
-		)
-		(pin "20"
-		)
-		(pin "1"
-		)
-		(pin "3"
-		)
-		(pin "2"
-		)
-		(instances
-			(project "CHeepCore"
-				(path "/1a6f5452-e688-4341-937f-30ed63281f98"
-					(reference "U101")
-					(unit 1)
-				)
-			)
-		)
 	)
 	(symbol
@@
 					(unit 1)
 				)
+			)
+		)
+	)
+	(symbol
+		(lib_id "MCU_WCH_CH32V0:CH32V003FxPx")
+		(at 123.19 105.41 0)
+		(unit 1)
+		(exclude_from_sim no)
+		(in_bom yes)
+		(on_board yes)
+		(dnp no)
+		(fields_autoplaced yes)
+		(property "Reference" "U101"
+			(at 125.4551 85.09 0)
+			(effects
+				(font
+					(size 1.27 1.27)
+				)
+				(justify left)
+			)
+		)
+		(property "Value" "CH32V003FxPx"
+			(at 125.4551 87.63 0)
+			(effects
+				(font
+					(size 1.27 1.27)
+				)
+				(justify left)
+			)
+		)
+		(property "Footprint" "Package_SO:TSSOP-20_4.4x6.5mm_P0.65mm"
+			(at 121.92 105.41 0)
+			(effects
+				(font
+					(size 1.27 1.27)
+				)
+				(hide yes)
+			)
+		)
+		(property "Datasheet" "https://www.wch-ic.com/products/CH32V003.html"
+			(at 121.92 105.41 0)
+			(effects
+				(font
+					(size 1.27 1.27)
+				)
+				(hide yes)
+			)
+		)
+		(property "Description" "CH32V003 series are industrial-grade general-purpose microcontrollers designed based on 32-bit RISC-V instruction set and architecture. It adopts QingKe V2A core, RV32EC instruction set, and supports 2 levels of interrupt nesting. The series are mounted with rich peripheral interfaces and function modules. Its internal organizational structure meets the low-cost and low-power embedded application scenarios."
+			(at 123.19 105.41 0)
+			(effects
+				(font
+					(size 1.27 1.27)
+				)
+				(hide yes)
+			)
+		)
+		(property "LCSC" "https://www.lcsc.com/product-detail/C5187096.html"
+			(at 123.19 105.41 0)
+			(effects
+				(font
+					(size 1.27 1.27)
+				)
+				(hide yes)
+			)
+		)
+		(property "Price @ 1000" "0.1349 €"
+			(at 123.19 105.41 0)
+			(effects
+				(font
+					(size 1.27 1.27)
+				)
+				(hide yes)
+			)
+		)
+		(pin "3"
+		)
+		(pin "15"
+		)
+		(pin "8"
+		)
+		(pin "10"
+		)
+		(pin "13"
+		)
+		(pin "11"
+		)
+		(pin "14"
+		)
+		(pin "16"
+		)
+		(pin "17"
+		)
+		(pin "18"
+		)
+		(pin "20"
+		)
+		(pin "19"
+		)
+		(pin "1"
+		)
+		(pin "9"
+		)
+		(pin "7"
+		)
+		(pin "2"
+		)
+		(pin "4"
+		)
+		(pin "5"
+		)
+		(pin "6"
+		)
+		(pin "12"
+		)
+		(instances
+			(project ""
+				(path "/1a6f5452-e688-4341-937f-30ed63281f98"
+					(reference "U101")
+					(unit 1)
+				)
